File: ethernet.kicad_sch (KiCad schematic)
At the start: 26 parts, among them J18 RJ45_LED, U7 ENC28J60x-SS, Y2 25 MHz

Commit message: Second version
Parts:
- removed C39, C40: 100n, Capacitor_SMD:C_0201_0603Metric_Pad0.64x0.40mm_HandSolder, symbol Device:C
- removed C41: 1n, Capacitor_SMD:C_0201_0603Metric_Pad0.64x0.40mm_HandSolder, symbol Device:C
- removed J18: RJ45_LED, Connector_RJ:RJ45_Amphenol_RJHSE538X, symbol Connector:RJ45_LED
- removed L5: L_Ferrite, Inductor_SMD:L_0805_2012Metric_Pad1.15x1.40mm_HandSolder, symbol Device:L_Ferrite
- removed RN2: R_Pack04, Resistor_SMD:R_Array_Convex_4x0612, symbol Device:R_Pack04
- removed RN3: 75, Resistor_SMD:R_Array_Convex_4x0612, symbol Device:R_Pack04
- removed TR1: WE_LAN_TRANSF_7490100110A, footprints:LAN Ethernet Wurth Elektronik, symbol myLibrary:WE_LAN_TRANSF_7490100110A
- R3: renamed from R28; footprint Resistor_SMD:R_0201_0603Metric_Pad0.64x0.40mm_HandSolder -> Resistor_SMD:R_0603_1608Metric_Pad0.98x0.95mm_HandSolder
- R4: renamed from R29; footprint Resistor_SMD:R_0201_0603Metric_Pad0.64x0.40mm_HandSolder -> Resistor_SMD:R_0603_1608Metric_Pad0.98x0.95mm_HandSolder
- R5: renamed from R30; footprint Resistor_SMD:R_0201_0603Metric_Pad0.64x0.40mm_HandSolder -> Resistor_SMD:R_0603_1608Metric_Pad0.98x0.95mm_HandSolder
- renumbered C36 to C10, C37 to C11, C38 to C12, C28 to C2, C29 to C3, C30 to C4, C31 to C5, C32 to C6, C33 to C7, C34 to C8, C35 to C9, L4 to L1, U7 to U1, Y2 to Y1
Connections:
- net ETH_FDX renamed LEDA
- net ETH_LINK renamed LEDB
- no-connect marks 3 -> 2
