File: power.kicad_sch (KiCad schematic)
At the start: 24 parts, among them T1 Transformer_1P_2S, U5 AP5100, U6 ZLDO1117K33TC

Commit message: Second version
Parts:
- renumbered C15 to C?, C14 to C?, C12 to C?, C10 to C?, C9 to C?, C13 to C?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
