File: radiator.kicad_sch (KiCad schematic)
At the start: 18 parts, among them J10 DS18B20, J11 Fluxmeter, J12 Electrovalve, J5 DS18B20, J6 DS18B20, J7 Fluxmeter, J8 Electrovalve, J9 DS18B20, Q2 Q_NPN_BCE, Q3 Q_NPN_BCE

Commit message: Second version
Parts:
- removed C6, C7, C8: C, Capacitor_SMD:C_0603_1608Metric_Pad1.08x0.95mm_HandSolder, symbol Device:C
- removed J10, J6, J9: DS18B20, Connector_JST:JST_PH_B3B-PH-K_1x03_P2.00mm_Vertical, symbol Connector_Generic:Conn_01x03
- J12: renamed from J11; footprint TerminalBlock_Phoenix:TerminalBlock_Phoenix_PT-1,5-2-3.5-H_1x02_P3.50mm_Horizontal -> Connector_JST:JST_PH_B2B-PH-K_1x02_P2.00mm_Vertical
- J9: renamed from J7; footprint TerminalBlock_Phoenix:TerminalBlock_Phoenix_PT-1,5-2-3.5-H_1x02_P3.50mm_Horizontal -> Connector_JST:JST_PH_B2B-PH-K_1x02_P2.00mm_Vertical
- R1: renamed from R11; footprint Resistor_SMD:R_0201_0603Metric_Pad0.64x0.40mm_HandSolder -> Resistor_SMD:R_0603_1608Metric_Pad0.98x0.95mm_HandSolder
- R2: renamed from R12; footprint Resistor_SMD:R_0201_0603Metric_Pad0.64x0.40mm_HandSolder -> Resistor_SMD:R_0603_1608Metric_Pad0.98x0.95mm_HandSolder
- renumbered C5 to C1, D3 to D1, D4 to D2, J8 to J10, J5 to J11, J12 to J13, Q2 to Q1, Q3 to Q2
Connections:
- net Electrovalve_switch2: no longer R2.1
- net Cold_Temp_Data1 renamed RADIATORS_REMP
Other:
- moved on the sheet: C1, J11
