File: smarthomeswitch.kicad_sch (KiCad schematic)
At the start: 56 parts, among them J1 Display, J15 USB_B_Micro, J17 Conn_ARM_JTAG_SWD_10, J2 Conn_01x03_Male, J3 PIR_SR505, J4 Conn_01x04_Male, K1 IM06, Q1 Q_NPN_BCE, U1 DS18B20, U2 ATSAM4S2AA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

Commit message: Second version
Parts:
- removed C1, C18: 10u, Capacitor_Tantalum_SMD:CP_EIA-3528-12_Kemet-T_Pad1.50x2.35mm_HandSolder, symbol Device:C
- removed C17: 100u, Capacitor_Tantalum_SMD:CP_EIA-6032-15_Kemet-U_Pad2.25x2.35mm_HandSolder, symbol Device:C
- removed C19, C20, C21, C22, C23, C24: 100n, Capacitor_SMD:C_0603_1608Metric_Pad1.08x0.95mm_HandSolder, symbol Device:C
- removed C2, C25, C26, C27, C3, C4: C, Capacitor_SMD:C_0603_1608Metric_Pad1.08x0.95mm_HandSolder, symbol Device:C
- removed D1: D_Schottky, Diode_SMD:D_Powermite2_AK, symbol Device:D_Schottky
- removed D2: DIODE, Diode_SMD:D_MELF_Handsoldering, symbol myLibrary:DIODE
- removed FB2, FB3: FerriteBead, Inductor_SMD:L_0603_1608Metric_Pad1.05x0.95mm_HandSolder, symbol Device:FerriteBead
- removed J1: Display, Connector_JST:JST_PH_B4B-PH-K_1x04_P2.00mm_Vertical, symbol Connector:Conn_01x04_Male
- removed J15: USB_B_Micro, Connector_USB:USB_Micro-B_Molex_47346-0001, symbol Connector:USB_B_Micro
- removed J17: Conn_ARM_JTAG_SWD_10, Connector_PinHeader_2.54mm:PinHeader_2x05_P2.54mm_Vertical, symbol Connector:Conn_ARM_JTAG_SWD_10
- removed J2: Conn_01x03_Male, TerminalBlock_Phoenix:TerminalBlock_Phoenix_MKDS-1,5-3-5.08_1x03_P5.08mm_Horizontal, symbol Connector:Conn_01x03_Male
- removed J3: PIR_SR505, Connector_PinHeader_2.54mm:PinHeader_1x03_P2.54mm_Vertical, symbol Connector_Generic:Conn_01x03
- removed J4: Conn_01x04_Male, TerminalBlock_Phoenix:TerminalBlock_Phoenix_MKDS-1,5-4-5.08_1x04_P5.08mm_Horizontal, symbol Connector:Conn_01x04_Male
- removed JP1, JP2, JP3: SolderJumper_2_Open, Jumper:SolderJumper-2_P1.3mm_Open_TrianglePad1.0x1.5mm, symbol Jumper:SolderJumper_2_Open
- removed K1: IM06, footprints:IM06CTS, symbol Relay:IM06
- removed L1: L, Inductor_SMD:L_Wuerth_WE-PD2-Typ-L, symbol Device:L
- removed Q1: Q_NPN_BCE, Package_TO_SOT_SMD:SOT-223-3_TabPin2, symbol Device:Q_NPN_BCE
- removed R1, R23, R24, R25, R26, R27, R32: 100, Resistor_SMD:R_0201_0603Metric_Pad0.64x0.40mm_HandSolder, symbol Device:R
- removed R10, R3, R4, R5, R6, R7, R9: R, Resistor_SMD:R_0201_0603Metric_Pad0.64x0.40mm_HandSolder, symbol Device:R
- removed R2, R22: 10k, Resistor_SMD:R_0201_0603Metric_Pad0.64x0.40mm_HandSolder, symbol Device:R
- removed R21: 4.02, Resistor_SMD:R_0201_0603Metric_Pad0.64x0.40mm_HandSolder, symbol Device:R
- removed R8: LDR03, Connector_PinHeader_2.54mm:PinHeader_1x02_P2.54mm_Vertical, symbol Sensor_Optical:LDR03
- removed RV1: R_Potentiometer, footprints:Potentiometer_Bourns_PTV09A-2_Single_Horizontal, symbol Device:R_Potentiometer
- removed RV2: R_Potentiometer, Potentiometer_SMD:Potentiometer_Bourns_TC33X_Vertical, symbol Device:R_Potentiometer
- removed U1: DS18B20, Package_TO_SOT_THT:TO-92_Inline, symbol Sensor_Temperature:DS18B20
- removed U2: ATSAM4S2AA, Package_QFP:LQFP-48_7x7mm_P0.5mm, symbol myLibrary:ATSAM4S2AA
- removed U3: LM3410, Package_TO_SOT_SMD:SOT-23-5_HandSoldering, symbol myLibrary:LM3410
- removed U4: LM358, Package_SO:SOIC-8_3.9x4.9mm_P1.27mm, symbol Amplifier_Operational:LM358
- removed Y1: 12/16 MHz, Crystal:Crystal_SMD_5032-4Pin_5.0x3.2mm, symbol Device:Crystal_GND24_Small
- added H1, H2, H3: MountingHole, MountingHole:MountingHole_3.2mm_M3_ISO14580, symbol Mechanical:MountingHole
Connections:
- no-connect marks 7 -> 0
Other:
- removed sheet Radiator
- removed sheet Windows
- removed sheet ethernet
- removed sheet power
- removed sheet touchkey
- added sheet BOTTOM PCB (main_power.kicad_sch)
- added sheet TOP PCB (core.kicad_sch)
- note added: "RJ45 VERTICAL: 735-0232"
