File: touchkey.kicad_sch (KiCad schematic)
At the start: 9 parts, among them U8 MTCH101

Commit message: Second version
Parts:
- R32: renamed from R16; footprint Resistor_SMD:R_0201_0603Metric_Pad0.64x0.40mm_HandSolder -> Resistor_SMD:R_0603_1608Metric_Pad0.98x0.95mm_HandSolder
- R33: renamed from R17; footprint Resistor_SMD:R_0201_0603Metric_Pad0.64x0.40mm_HandSolder -> Resistor_SMD:R_0603_1608Metric_Pad0.98x0.95mm_HandSolder
- R34: renamed from R18; footprint Resistor_SMD:R_0201_0603Metric_Pad0.64x0.40mm_HandSolder -> Resistor_SMD:R_0603_1608Metric_Pad0.98x0.95mm_HandSolder
- R35: renamed from R19; footprint Resistor_SMD:R_0201_0603Metric_Pad0.64x0.40mm_HandSolder -> Resistor_SMD:R_0603_1608Metric_Pad0.98x0.95mm_HandSolder
- R36: renamed from R20; footprint Resistor_SMD:R_0201_0603Metric_Pad0.64x0.40mm_HandSolder -> Resistor_SMD:R_0603_1608Metric_Pad0.98x0.95mm_HandSolder
- renumbered C16 to C37, RV3 to RV2
Connections:
- net VDD renamed +3V3
Other:
- note added: "VDD: voltage will give the lowest sensitivity GND: voltage will give the highest sensitivity"
Changed lines of the file:
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@@
     (stroke (width 0) (type default) (color 0 0 0 0))
+  )
+  (text "VDD: voltage will give the lowest sensitivity\nGND: voltage will give the highest sensitivity"
+    (at 43.815 70.485 90)
+    (effects (font (size 1.27 1.27)) (justify left bottom))
   )
   (hierarchical_label "TouchKeySwitch" (shape input) (at 85.09 60.325 0)
@@
   (symbol (lib_id "myLibrary:GND") (at 65.405 45.72 270) (unit 1)
     (in_bom yes) (on_board yes) (fields_autoplaced)
-    (property "Reference" "#PWR056" (id 0) (at 59.055 45.72 0)
+    (property "Reference" "#PWR098" (id 0) (at 59.055 45.72 0)
       (effects (font (size 1.27 1.27)) hide)
     )
@@
   (symbol (lib_id "Device:R") (at 60.325 49.53 90) (unit 1)
     (in_bom yes) (on_board yes)
-    (property "Reference" "R17" (id 0) (at 60.325 51.435 90))
+    (property "Reference" "R33" (id 0) (at 60.325 51.435 90))
     (property "Value" "10k" (id 1) (at 60.325 47.3511 90))
-    (property "Footprint" "Resistor_SMD:R_0201_0603Metric_Pad0.64x0.40mm_HandSolder" (id 2) (at 60.325 51.308 90)
+    (property "Footprint" "Resistor_SMD:R_0603_1608Metric_Pad0.98x0.95mm_HandSolder" (id 2) (at 60.325 51.308 90)
       (effects (font (size 1.27 1.27)) hide)
     )
@@
     (pin "1")
     (pin "2")
+  )
+  (symbol (lib_id "myLibrary:+3V3") (at 47.625 41.91 0) (unit 1)
+    (in_bom yes) (on_board yes) (fields_autoplaced)
+    (property "Reference" "#PWR0118" (id 0) (at 47.625 45.72 0)
+      (effects (font (size 1.27 1.27)) hide)
+    )
+    (property "Value" "+3V3" (id 1) (at 47.625 38.3342 0))
+    (property "Footprint" "" (id 2) (at 47.625 41.91 0))
+    (property "Datasheet" "" (id 3) (at 47.625 41.91 0))
+    (pin "1")
   )
   (symbol (lib_id "Device:R") (at 61.595 40.64 90) (unit 1)
     (in_bom yes) (on_board yes)
-    (property "Reference" "R18" (id 0) (at 61.595 42.545 90))
+    (property "Reference" "R34" (id 0) (at 61.595 42.545 90))
     (property "Value" "4k7" (id 1) (at 61.595 38.4611 90))
-    (property "Footprint" "Resistor_SMD:R_0201_0603Metric_Pad0.64x0.40mm_HandSolder" (id 2) (at 61.595 42.418 90)
+    (property "Footprint" "Resistor_SMD:R_0603_1608Metric_Pad0.98x0.95mm_HandSolder" (id 2) (at 61.595 42.418 90)
       (effects (font (size 1.27 1.27)) hide)
     )
@@
     (pin "2")
   )
-  (symbol (lib_id "myLibrary:VDD") (at 93.98 34.29 0) (unit 1)
-    (in_bom yes) (on_board yes) (fields_autoplaced)
-    (property "Reference" "#PWR057" (id 0) (at 93.98 38.1 0)
-      (effects (font (size 1.27 1.27)) hide)
-    )
-    (property "Value" "VDD" (id 1) (at 93.98 30.7142 0))
-    (property "Footprint" "" (id 2) (at 93.98 34.29 0))
-    (property "Datasheet" "" (id 3) (at 93.98 34.29 0))
+  (symbol (lib_id "myLibrary:+3V3") (at 100.965 45.72 0) (unit 1)
+    (in_bom yes) (on_board yes) (fields_autoplaced)
+    (property "Reference" "#PWR0120" (id 0) (at 100.965 49.53 0)
+      (effects (font (size 1.27 1.27)) hide)
+    )
+    (property "Value" "+3V3" (id 1) (at 100.965 42.1442 0))
+    (property "Footprint" "" (id 2) (at 100.965 45.72 0))
+    (property "Datasheet" "" (id 3) (at 100.965 45.72 0))
     (pin "1")
   )
   (symbol (lib_id "Device:R") (at 47.625 45.72 0) (unit 1)
     (in_bom yes) (on_board yes) (fields_autoplaced)
-    (property "Reference" "R16" (id 0) (at 49.403 44.8853 0)
+    (property "Reference" "R32" (id 0) (at 49.403 44.8853 0)
       (effects (font (size 1.27 1.27)) (justify left))
     )
@@
       (effects (font (size 1.27 1.27)) (justify left))
     )
-    (property "Footprint" "Resistor_SMD:R_0201_0603Metric_Pad0.64x0.40mm_HandSolder" (id 2) (at 45.847 45.72 90)
+    (property "Footprint" "Resistor_SMD:R_0603_1608Metric_Pad0.98x0.95mm_HandSolder" (id 2) (at 45.847 45.72 90)
       (effects (font (size 1.27 1.27)) hide)
     )
@@
   (symbol (lib_id "Device:R") (at 84.455 55.245 0) (unit 1)
     (in_bom yes) (on_board yes) (fields_autoplaced)
-    (property "Reference" "R19" (id 0) (at 86.233 54.4103 0)
+    (property "Reference" "R35" (id 0) (at 86.233 54.4103 0)
       (effects (font (size 1.27 1.27)) (justify left))
     )
@@
       (effects (font (size 1.27 1.27)) (justify left))
     )
-    (property "Footprint" "Resistor_SMD:R_0201_0603Metric_Pad0.64x0.40mm_HandSolder" (id 2) (at 82.677 55.245 90)
+    (property "Footprint" "Resistor_SMD:R_0603_1608Metric_Pad0.98x0.95mm_HandSolder" (id 2) (at 82.677 55.245 90)
       (effects (font (size 1.27 1.27)) hide)
     )
@@
   (symbol (lib_id "Device:R_Potentiometer") (at 47.625 53.975 0) (unit 1)
     (in_bom yes) (on_board yes) (fields_autoplaced)
-    (property "Reference" "RV3" (id 0) (at 45.8471 53.1403 0)
+    (property "Reference" "RV2" (id 0) (at 45.8471 53.1403 0)
       (effects (font (size 1.27 1.27)) (justify right))
     )
@@
   (symbol (lib_id "myLibrary:GND") (at 96.52 53.34 0) (unit 1)
     (in_bom yes) (on_board yes) (fields_autoplaced)
-    (property "Reference" "#PWR058" (id 0) (at 96.52 59.69 0)
+    (property "Reference" "#PWR0100" (id 0) (at 96.52 59.69 0)
       (effects (font (size 1.27 1.27)) hide)
     )
@@
   (symbol (lib_id "Device:C") (at 96.52 49.53 0) (unit 1)
     (in_bom yes) (on_board yes) (fields_autoplaced)
-    (property "Reference" "C16" (id 0) (at 99.441 48.6953 0)
+    (property "Reference" "C37" (id 0) (at 99.441 48.6953 0)
       (effects (font (size 1.27 1.27)) (justify left))
     )
@@
     (pin "2")
   )
+  (symbol (lib_id "myLibrary:+3V3") (at 93.98 34.29 0) (unit 1)
+    (in_bom yes) (on_board yes) (fields_autoplaced)
+    (property "Reference" "#PWR0119" (id 0) (at 93.98 38.1 0)
+      (effects (font (size 1.27 1.27)) hide)
+    )
+    (property "Value" "+3V3" (id 1) (at 93.98 30.7142 0))
+    (property "Footprint" "" (id 2) (at 93.98 34.29 0))
+    (property "Datasheet" "" (id 3) (at 93.98 34.29 0))
+    (pin "1")
+  )
   (symbol (lib_id "myLibrary:GND") (at 47.625 59.055 0) (unit 1)
     (in_bom yes) (on_board yes) (fields_autoplaced)
-    (property "Reference" "#PWR055" (id 0) (at 47.625 65.405 0)
+    (property "Reference" "#PWR097" (id 0) (at 47.625 65.405 0)
       (effects (font (size 1.27 1.27)) hide)
     )
@@
   (symbol (lib_id "Device:R") (at 93.98 38.1 0) (unit 1)
     (in_bom yes) (on_board yes) (fields_autoplaced)
-    (property "Reference" "R20" (id 0) (at 95.758 37.2653 0)
+    (property "Reference" "R36" (id 0) (at 95.758 37.2653 0)
       (effects (font (size 1.27 1.27)) (justify left))
     )
@@
       (effects (font (size 1.27 1.27)) (justify left))
     )
-    (property "Footprint" "Resistor_SMD:R_0201_0603Metric_Pad0.64x0.40mm_HandSolder" (id 2) (at 92.202 38.1 90)
+    (property "Footprint" "Resistor_SMD:R_0603_1608Metric_Pad0.98x0.95mm_HandSolder" (id 2) (at 92.202 38.1 90)
       (effects (font (size 1.27 1.27)) hide)
     )
@@
     (pin "6")
   )
-  (symbol (lib_id "myLibrary:VDD") (at 47.625 41.91 0) (unit 1)
-    (in_bom yes) (on_board yes) (fields_autoplaced)
-    (property "Reference" "#PWR0143" (id 0) (at 47.625 45.72 0)
-      (effects (font (size 1.27 1.27)) hide)
-    )
-    (property "Value" "VDD" (id 1) (at 47.625 38.3342 0))
-    (property "Footprint" "" (id 2) (at 47.625 41.91 0))
-    (property "Datasheet" "" (id 3) (at 47.625 41.91 0))
-    (pin "1")
-  )
-  (symbol (lib_id "myLibrary:VDD") (at 100.965 45.72 0) (unit 1)
-    (in_bom yes) (on_board yes) (fields_autoplaced)
-    (property "Reference" "#PWR059" (id 0) (at 100.965 49.53 0)
-      (effects (font (size 1.27 1.27)) hide)
-    )
-    (property "Value" "VDD" (id 1) (at 100.965 42.1442 0))
-    (property "Footprint" "" (id 2) (at 100.965 45.72 0))
-    (property "Datasheet" "" (id 3) (at 100.965 45.72 0))
-    (pin "1")
-  )
 )
