File: windows.kicad_sch (KiCad schematic)
At the start: 1 part, among them J13 Conn_01x04_Male

Commit message: Second version
Parts:
- renumbered J13 to J14
Changed lines of the file:
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@@
   (symbol (lib_id "Connector:Conn_01x04_Male") (at 76.835 28.575 180) (unit 1)
     (in_bom yes) (on_board yes) (fields_autoplaced)
-    (property "Reference" "J13" (id 0) (at 77.5462 26.4703 0)
+    (property "Reference" "J14" (id 0) (at 77.5462 26.4703 0)
       (effects (font (size 1.27 1.27)) (justify right))
     )
@@
   (symbol (lib_id "myLibrary:GND") (at 71.755 31.115 0) (unit 1)
     (in_bom yes) (on_board yes) (fields_autoplaced)
-    (property "Reference" "#PWR0142" (id 0) (at 71.755 37.465 0)
+    (property "Reference" "#PWR031" (id 0) (at 71.755 37.465 0)
       (effects (font (size 1.27 1.27)) hide)
     )
